File: pico-can.kicad_pcb (KiCad board)
At the start: 2 copper layers, 22.9 x 50.8 mm, 71 parts, among them J1 USB_C_Receptacle_USB2.0, J2 I2C, J3 Screw_Terminal_01x03, J4 Conn, J5 Conn, J6 BAT, Q1 BSS83P, SW1 SW_Push, SW2 SW_Push, U1 RP2040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

Commit message: add screen shoot image
Routing:
- net VBUS: track 0.00 -> 55.6 mm, vias 0 -> 6
- net /GPIO13: track 0.00 -> 27.3 mm, vias 0 -> 2
- net VBAT: track 0.00 -> 24.2 mm
- net +3V3: track 4.65 -> 24.6 mm
- net VHI: track 0.00 -> 19.8 mm, vias 0 -> 2
- net /GPIO9: track 0.00 -> 17.5 mm, vias 0 -> 1
- net /GPIO10: track 0.00 -> 15.4 mm, vias 0 -> 1
- net /GPIO11: track 0.00 -> 13.4 mm, vias 0 -> 1
- net /GPIO12: track 0.00 -> 12.5 mm, vias 0 -> 1
- net /GPIO26_ADC0: track 0.00 -> 11.9 mm
- net /GPIO27_ADC1: track 0.00 -> 9.86 mm
- net /QSPI_SD3: track 0.00 -> 9.85 mm
- net /~{RST}: track 0.00 -> 9.53 mm
- net /GPIO25: track 0.00 -> 9.08 mm, vias 0 -> 1
- net /QSPI_SCLK: track 0.00 -> 8.17 mm
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